File: pcb/esp32s3/esp32s3.kicad_pcb (KiCad board)
At the start: 2 copper layers, 0 parts

Commit message: updated footprints / schematic
Parts:
- added ATGM336H1: ~, footprints:ATGM336H, F.Cu at (111.3, 81.8)
- added BT1: MS421R, footprints:MSR421R, F.Cu at (152.5, 81.1)
- added C1: 10pF, Capacitor_SMD:C_0402_1005Metric, F.Cu at (121.0, 52.0)
- added C10: 100nF, Capacitor_SMD:C_0402_1005Metric, F.Cu at (126.7, 53.9)
- added C11: 100nF, Capacitor_SMD:C_0402_1005Metric, F.Cu at (126.7, 55.9)
- added C12: 10uF, Capacitor_SMD:C_0402_1005Metric, F.Cu at (126.7, 57.9)
- added C13: 10uF, Capacitor_SMD:C_0402_1005Metric, F.Cu at (148.2, 52.0)
- added C14: 22uF, Capacitor_SMD:C_0402_1005Metric, F.Cu at (148.2, 53.9)
- added C15: 10uF, Capacitor_SMD:C_0402_1005Metric, F.Cu at (118.3, 88.3)
- added C16: 100nF, Capacitor_SMD:C_0402_1005Metric, F.Cu at (118.3, 90.3)
- added C17: 1uF, Capacitor_SMD:C_0402_1005Metric, F.Cu at (134.5, 76.0)
- added C18: 100nF, Capacitor_SMD:C_0402_1005Metric, F.Cu at (134.5, 78.0)
- added C19: 1.8pF, Capacitor_SMD:C_0402_1005Metric, F.Cu at (134.5, 79.9)
- added C2: 2p4, Capacitor_SMD:C_0402_1005Metric, F.Cu at (121.0, 53.9)
- added C20: 47nF, Capacitor_SMD:C_0402_1005Metric, F.Cu at (134.5, 81.9)
- added C21: 470nF, Capacitor_SMD:C_0402_1005Metric, F.Cu at (137.4, 76.0)
- added C22: 2.4pF, Capacitor_SMD:C_0402_1005Metric, F.Cu at (137.4, 78.0)
- added C23: 47pF, Capacitor_SMD:C_0402_1005Metric, F.Cu at (137.4, 79.9)
- added C24: 3pF, Capacitor_SMD:C_0402_1005Metric, F.Cu at (137.4, 81.9)
- added C25: 5.6pF, Capacitor_SMD:C_0402_1005Metric, F.Cu at (140.3, 76.0)
- added C26: 3.3pF, Capacitor_SMD:C_0402_1005Metric, F.Cu at (140.3, 78.0)
- added C27: 39pF, Capacitor_SMD:C_0402_1005Metric, F.Cu at (140.3, 79.9)
- added C28: 3.3pF, Capacitor_SMD:C_0402_1005Metric, F.Cu at (140.3, 81.9)
- added C29: 1.8pF, Capacitor_SMD:C_0402_1005Metric, F.Cu at (143.1, 76.0)
- added C3: 100nF, Capacitor_SMD:C_0402_1005Metric, F.Cu at (121.0, 55.9)
- added C30: 39pF, Capacitor_SMD:C_0402_1005Metric, F.Cu at (143.1, 78.0)
- added C31: 1nF, Capacitor_SMD:C_0402_1005Metric, F.Cu at (143.1, 79.9)
- added C32: 1nF, Capacitor_SMD:C_0402_1005Metric, F.Cu at (143.1, 81.9)
- added C33: 220nF, Capacitor_SMD:C_0402_1005Metric, F.Cu at (126.1, 77.2)
- added C4: 2p7, Capacitor_SMD:C_0402_1005Metric, F.Cu at (121.0, 57.9)
- added C5: 10pF, Capacitor_SMD:C_0402_1005Metric, F.Cu at (123.9, 52.0)
- added C6: 10uF, Capacitor_SMD:C_0402_1005Metric, F.Cu at (123.9, 53.9)
- added C7: 0.1uF, Capacitor_SMD:C_0402_1005Metric, F.Cu at (123.9, 55.9)
- added C8: 0.1uF, Capacitor_SMD:C_0402_1005Metric, F.Cu at (123.9, 57.9)
- added C9: 0.1uF, Capacitor_SMD:C_0402_1005Metric, F.Cu at (126.7, 52.0)
- added D1: MBR0540, Diode_SMD:D_SOD-123, F.Cu at (144.8, 57.3)
- added D2: MBR0540, Diode_SMD:D_SOD-123, F.Cu at (114.0, 89.0)
- added J1: USB_C_Receptacle_USB2.0_14P, Connector_USB:USB_C_Receptacle_G-Switch_GT-USB-7010ASV, F.Cu at (136.0, 56.4)
- added J2: Battery, footprints:2 Wire Pads, F.Cu at (132.2, 70.9)
- added J3: GPS_ANT, Connector_Coaxial:U.FL_Molex_MCRF_73412-0110_Vertical, F.Cu at (108.0, 90.4)
- added L1: 2n4, Inductor_SMD:L_0402_1005Metric, F.Cu at (118.1, 52.0)
- added L2: 2n2, Inductor_SMD:L_0402_1005Metric, F.Cu at (118.1, 54.0)
- added L3: 47nH, Inductor_SMD:L_0402_1005Metric, F.Cu at (112.5, 91.7)
- added L4: 15uH, Inductor_SMD:L_0402_1005Metric, F.Cu at (131.6, 76.0)
- added L5: 15nH, Inductor_SMD:L_0402_1005Metric, F.Cu at (131.6, 78.0)
- added L6: 47nH, Inductor_SMD:L_0402_1005Metric, F.Cu at (131.6, 80.0)
- added L7: 2.5nH, Inductor_SMD:L_0402_1005Metric, F.Cu at (131.6, 82.0)
- added L8: 9.1nH, Inductor_SMD:L_0402_1005Metric, F.Cu at (131.6, 84.0)
- added L9: 4.7nH, Inductor_SMD:L_0402_1005Metric, F.Cu at (131.6, 86.0)
- added Q1: DMG3414U, Package_TO_SOT_SMD:SOT-23, F.Cu at (144.3, 53.4)
- added Q1_Xtal1: 32.0MHz, Crystal:Crystal_SMD_2016-4Pin_2.0x1.6mm, F.Cu at (141.3, 90.8)
- added R1: 10k, Resistor_SMD:R_0402_1005Metric, F.Cu at (118.1, 56.0)
- added R10: 200k, Resistor_SMD:R_0402_1005Metric, F.Cu at (141.5, 70.0)
- added R11: 200k, Resistor_SMD:R_0402_1005Metric, F.Cu at (141.5, 72.0)
- added R12: 100R, Resistor_SMD:R_0402_1005Metric, F.Cu at (131.6, 87.9)
- added R13: 100R, Resistor_SMD:R_0402_1005Metric, F.Cu at (131.6, 89.9)
- added R14: 10K, Resistor_SMD:R_0402_1005Metric, F.Cu at (123.2, 77.2)
- added R15: 10K, Resistor_SMD:R_0402_1005Metric, F.Cu at (123.2, 79.2)
- added R16: 10K, Resistor_SMD:R_0402_1005Metric, F.Cu at (123.2, 81.1)
- added R17: 10K, Resistor_SMD:R_0402_1005Metric, F.Cu at (123.2, 83.1)
- added R18: 22, Resistor_SMD:R_0402_1005Metric, F.Cu at (146.2, 74.4)
- added R2: 5k1, Resistor_SMD:R_0402_1005Metric, F.Cu at (118.1, 58.0)
- added R3: 200k, Resistor_SMD:R_0402_1005Metric, F.Cu at (118.1, 59.9)
- added R4: 200k, Resistor_SMD:R_0402_1005Metric, F.Cu at (118.1, 61.9)
- added R5: 10k, Resistor_SMD:R_0402_1005Metric, F.Cu at (118.1, 63.9)
- added R6: 5.1k, Resistor_SMD:R_0402_1005Metric, F.Cu at (141.5, 62.1)
- added R7: 5.1k, Resistor_SMD:R_0402_1005Metric, F.Cu at (141.5, 64.0)
- added R8: 5.1k, Resistor_SMD:R_0402_1005Metric, F.Cu at (141.5, 66.0)
- added R9: 100k, Resistor_SMD:R_0402_1005Metric, F.Cu at (141.5, 68.0)
- added RFIO1: SMA, Connector_Coaxial:U.FL_Molex_MCRF_73412-0110_Vertical, F.Cu at (142.4, 85.9)
- added SW1: BOOT, Button_Switch_SMD:SW_MEC_5GSH9, F.Cu at (99.5, 47.6)
- added TP1: Reset, Connector_PinHeader_1.00mm:PinHeader_1x02_P1.00mm_Horizontal, F.Cu at (109.2, 60.9)
- added U1: ESP32-S3FN8, Package_DFN_QFN:QFN-56-1EP_7x7mm_P0.4mm_EP4x4mm, F.Cu at (121.3, 69.5)
- added U2: AZ1117-3.3, Package_TO_SOT_SMD:SOT-223-3_TabPin2, F.Cu at (135.1, 65.3)
- added U3: USBLC6-2SC6, Package_TO_SOT_SMD:SOT-23-6, F.Cu at (145.5, 63.5)
- added U4: MCP73831-2-OT, Package_TO_SOT_SMD:SOT-23-5, F.Cu at (145.5, 68.1)
- added U5: 24AA32AF-I_MS, KiCAD Parts:SOP65P490X110-8N, F.Cu at (152.9, 75.5)
- added U6: SX1262IMLTRT, Package_DFN_QFN:QFN-24-1EP_4x4mm_P0.5mm_EP2.6x2.6mm, F.Cu at (136.2, 86.0)
- added U7: PE4259, KiCAD Parts:SOT65P215X110-6N, F.Cu at (152.0, 88.8)
- added U8: LSM303AGR, KiCAD Parts:PQFN50P200X200X100-12N, F.Cu at (135.3, 93.8)
- added U9: 2450AT18D0100E, 2450AT18D0100E:2450AT18D0100E_JOT, F.Cu at (111.8, 54.4)
- added X1: 40MHz, Crystal:Crystal_SMD_Abracon_ABM10-4Pin_2.5x2.0mm, F.Cu at (107.1, 69.9)
Other:
- board outline added: 64.5 x 64.5 mm
