File: pcb/esp32s3/esp32s3.kicad_sch (KiCad schematic)
At the start: 24 parts, among them SW1 BOOT, U1 ESP32-S3FN8, X1 40MHz

Commit message: updated footprints / schematic
Parts:
- removed AE1: Antenna_Chip, symbol Device:Antenna_Chip
- added R18: 22, Resistor_SMD:R_0402_1005Metric, symbol Device:R_US
- added U9: 2450AT18D0100E, 2450AT18D0100E:2450AT18D0100E_JOT, symbol 2024-04-20_02-03-53:2450AT18D0100E
- C1: renamed from C11; footprint (none) -> Capacitor_SMD:C_0402_1005Metric
- C10: renamed from C5; footprint (none) -> Capacitor_SMD:C_0402_1005Metric
- C11: renamed from C6; footprint (none) -> Capacitor_SMD:C_0402_1005Metric
- C12: renamed from C7; footprint (none) -> Capacitor_SMD:C_0402_1005Metric
- C2: renamed from C10; value 3p3 -> 2p4; footprint (none) -> Capacitor_SMD:C_0402_1005Metric
- C3: renamed from C8; footprint (none) -> Capacitor_SMD:C_0402_1005Metric
- C4: renamed from C9; value 3p3 -> 2p7; footprint (none) -> Capacitor_SMD:C_0402_1005Metric
- C5: renamed from C12; footprint (none) -> Capacitor_SMD:C_0402_1005Metric
- C6: renamed from C1; footprint (none) -> Capacitor_SMD:C_0402_1005Metric
- C7: renamed from C2; footprint (none) -> Capacitor_SMD:C_0402_1005Metric
- C8: renamed from C3; footprint (none) -> Capacitor_SMD:C_0402_1005Metric
- C9: renamed from C4; footprint (none) -> Capacitor_SMD:C_0402_1005Metric
- L1: renamed from L2; value 2n2 -> 2n4; footprint (none) -> Inductor_SMD:L_0402_1005Metric
- L2: renamed from L1; footprint (none) -> Inductor_SMD:L_0402_1005Metric
- R1, R2: footprint (none) -> Resistor_SMD:R_0402_1005Metric
- R3: renamed from R11; footprint (none) -> Resistor_SMD:R_0402_1005Metric
- R4: renamed from R8; footprint (none) -> Resistor_SMD:R_0402_1005Metric
- R5: renamed from R3; footprint (none) -> Resistor_SMD:R_0402_1005Metric
- X1: footprint (none) -> Crystal:Crystal_SMD_Abracon_ABM10-4Pin_2.5x2.0mm
Connections:
- net GND: now also U9.2 (GND), U9.3 (GND), U9.4 (GND/FEED)
- net XTAL_P: now also R18.1; no longer C1.1, X1.1
- net at C2.1, L1.2: now also U9.1 (FEED/GND)
- net GP10 renamed INT_MAG
- net GP11 renamed XL_INT0
- net GP12 renamed XL_INT1
- net GP13 renamed LoRa_MISO
- net GP14 renamed LoRa_MOSI
- net GP17 renamed LoRa_NSS
- net GP18 renamed LoRa_SCK
- net GP21 renamed LoRa_RST
- net GP3: no longer names the net of U1.8 (GPIO3)
- net GP4 renamed GPS_TXD
- net GP43 renamed LoRa_DIO1
- net GP44 renamed LoRa_BUSY
- net GP5 renamed GPS_RXD
- net GP6 renamed GPS_ON
- net GPS_ON: now also U1.12 (GPIO7); no longer U1.11 (GPIO6)
- net GP7 renamed GPS_RESET
- net GPS_RESET: now also U1.11 (GPIO6); no longer U1.12 (GPIO7)
- net GP8 renamed XL_COMP_SCL
- net GP9 renamed XL_COMP_SDA
- new net: C1.1, R18.2, X1.1
- no-connect marks 10 -> 11
Other:
- added sheet Accel & Magnetometer (untitled.kicad_sch)
- added sheet LoRa (festitracker.kicad_sch)
- note added: "Accel & Magnetometer"
- note added: "LoRa Circuit"
- note added: "Power & USB"
- moved on the sheet: C1, C2, C4, C5, L1, R1, R3, R4, TP1, X1

Commit message: pcb update!!!
Parts:
- added J4: LH128R-IG01, LH128R-IG01:LH128R-IG01, symbol LH128R-IG01:LH128R-IG01
- added Q2: DMG1012T, Package_TO_SOT_SMD:SOT-523, symbol Transistor_FET:DMG1012T
- added R19: 10, Resistor_SMD:R_0402_1005Metric, symbol Device:R_US
- added R20: 10K, Resistor_SMD:R_0402_1005Metric, symbol Device:R_US
- added R21: 1K, Resistor_SMD:R_0402_1005Metric, symbol Device:R_US
- C2: value 2p4 -> 2.4pF
- C4: value 2p7 -> 2.7pF
- C7, C8, C9: value 0.1uF -> 100nF
- L1: value 2n4 -> 2.4nH
Connections:
- net GND: now also J4.1 (GND), J4.12 (GND), J4.5 (GND), J4.6 (GND), Q2.2 (S), R20.1
- net GP37 renamed LCD_BL
- net LCD_BL: now also R21.1
- net GP38 renamed LCD_DC
- net LCD_DC: now also J4.7 (D/C)
- net GP39 renamed LCD_CS
- net LCD_CS: now also J4.8 (CS)
- net GP40 renamed LCD_SCK
- net LCD_SCK: now also J4.9 (SCL)
- net GP41 renamed LCD_SDA
- net LCD_SDA: now also J4.10 (SDA)
- net GP42 renamed LCD_RST
- net LCD_RST: now also J4.11 (RESET)
- new net: Q2.1 (G), R20.2, R21.2
- new net: Q2.3 (D), R19.2
- new net: J4.2 (LEDK), R19.1
- new net VDD: J4.3 (LEDA), J4.4 (VDD)
