File: pcb/esp32s3/gps.kicad_sch (KiCad schematic)
At the start: 8 parts, among them J3 GPS_ANT, U5 24AA32AF-I_MS

Commit message: updated footprints / schematic
Parts:
- BT1: footprint (none) -> footprints:MSR421R
- C15, C16: footprint (none) -> Capacitor_SMD:C_0402_1005Metric
- L3: footprint (none) -> Inductor_SMD:L_0402_1005Metric
- U5: footprint 24AA32AF-I_MS:SOP65P490X110-8N -> KiCAD Parts:SOP65P490X110-8N
- renumbered ATGM336H2 to ATGM336H1
Changed lines of the file:
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@@
 			)
 		)
-		(property "Footprint" ""
+		(property "Footprint" "Capacitor_SMD:C_0402_1005Metric"
 			(at 129.2352 49.53 0)
 			(effects
@@
 			)
 		)
-		(property "Footprint" ""
+		(property "Footprint" "footprints:MSR421R"
 			(at 193.04 73.406 90)
 			(effects
@@
 			)
 		)
-		(property "Footprint" "24AA32AF-I_MS:SOP65P490X110-8N"
+		(property "Footprint" "KiCAD Parts:SOP65P490X110-8N"
 			(at 86.36 97.79 0)
 			(effects
@@
 		(dnp no)
 		(fields_autoplaced yes)
-		(property "Reference" "#PWR034"
+		(property "Reference" "#PWR041"
 			(at 193.04 58.42 0)
 			(effects
@@
 			(project "esp32s3"
 				(path "/834edf73-57a5-43b4-ab36-0b077e93e6d5/c241b7c0-effc-4bf6-a5ff-9f24a08e0fe4"
-					(reference "#PWR034")
+					(reference "#PWR041")
 					(unit 1)
 				)
@@
 		(dnp no)
 		(fields_autoplaced yes)
-		(property "Reference" "#PWR037"
+		(property "Reference" "#PWR035"
 			(at 60.96 106.68 0)
 			(effects
@@
 			(project "esp32s3"
 				(path "/834edf73-57a5-43b4-ab36-0b077e93e6d5/c241b7c0-effc-4bf6-a5ff-9f24a08e0fe4"
-					(reference "#PWR037")
+					(reference "#PWR035")
 					(unit 1)
 				)
@@
 		(on_board yes)
 		(dnp no)
-		(property "Reference" "ATGM336H2"
-			(at 138.43 57.15 0)
+		(property "Reference" "ATGM336H1"
+			(at 138.43 55.118 0)
 			(effects
 				(font
@@
 			(project "esp32s3"
 				(path "/834edf73-57a5-43b4-ab36-0b077e93e6d5/c241b7c0-effc-4bf6-a5ff-9f24a08e0fe4"
-					(reference "ATGM336H2")
+					(reference "ATGM336H1")
 					(unit 1)
 				)
@@
 		(on_board yes)
 		(dnp no)
-		(property "Reference" "#PWR036"
+		(property "Reference" "#PWR037"
 			(at 104.14 76.2 0)
 			(effects
@@
 			(project "esp32s3"
 				(path "/834edf73-57a5-43b4-ab36-0b077e93e6d5/c241b7c0-effc-4bf6-a5ff-9f24a08e0fe4"
-					(reference "#PWR036")
+					(reference "#PWR037")
 					(unit 1)
 				)
@@
 		(dnp no)
 		(fields_autoplaced yes)
-		(property "Reference" "#PWR038"
+		(property "Reference" "#PWR036"
 			(at 64.77 115.57 0)
 			(effects
@@
 			(project "esp32s3"
 				(path "/834edf73-57a5-43b4-ab36-0b077e93e6d5/c241b7c0-effc-4bf6-a5ff-9f24a08e0fe4"
-					(reference "#PWR038")
+					(reference "#PWR036")
 					(unit 1)
 				)
@@
 			)
 		)
-		(property "Footprint" ""
+		(property "Footprint" "Capacitor_SMD:C_0402_1005Metric"
 			(at 147.0152 49.53 0)
 			(effects
@@
 		(on_board yes)
 		(dnp no)
-		(property "Reference" "#PWR032"
+		(property "Reference" "#PWR039"
 			(at 137.16 55.88 0)
 			(effects
@@
 			(project "esp32s3"
 				(path "/834edf73-57a5-43b4-ab36-0b077e93e6d5/c241b7c0-effc-4bf6-a5ff-9f24a08e0fe4"
-					(reference "#PWR032")
+					(reference "#PWR039")
 					(unit 1)
 				)
@@
 		(dnp no)
 		(fields_autoplaced yes)
-		(property "Reference" "#PWR035"
+		(property "Reference" "#PWR042"
 			(at 193.04 87.63 0)
 			(effects
@@
 			(project "esp32s3"
 				(path "/834edf73-57a5-43b4-ab36-0b077e93e6d5/c241b7c0-effc-4bf6-a5ff-9f24a08e0fe4"
-					(reference "#PWR035")
+					(reference "#PWR042")
 					(unit 1)
 				)
@@
 			)
 		)
-		(property "Footprint" ""
+		(property "Footprint" "Inductor_SMD:L_0402_1005Metric"
 			(at 118.11 71.12 0)
 			(effects
@@
 		(dnp no)
 		(fields_autoplaced yes)
-		(property "Reference" "#PWR033"
+		(property "Reference" "#PWR038"
 			(at 137.16 43.18 0)
 			(effects
@@
 			(project "esp32s3"
 				(path "/834edf73-57a5-43b4-ab36-0b077e93e6d5/c241b7c0-effc-4bf6-a5ff-9f24a08e0fe4"
-					(reference "#PWR033")
+					(reference "#PWR038")
 					(unit 1)
 				)
@@
 		(dnp no)
 		(fields_autoplaced yes)
-		(property "Reference" "#PWR031"
+		(property "Reference" "#PWR040"
 			(at 154.94 96.52 0)
 			(effects
@@
 			(project "esp32s3"
 				(path "/834edf73-57a5-43b4-ab36-0b077e93e6d5/c241b7c0-effc-4bf6-a5ff-9f24a08e0fe4"
-					(reference "#PWR031")
-					(unit 1)
-				)
+					(reference "#PWR040")
+					(unit 1)
+				)

Commit message: Update PCB with new components and footprints
Parts:
- ATGM336H1: footprint footprints:ATGM336H -> custom_comps:ATGM336H
- BT1: footprint footprints:MSR421R -> custom_comps:MSR421R
- U5: footprint KiCAD Parts:SOP65P490X110-8N -> custom_comps:SOP65P490X110-8N
Changed lines of the file:
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@@
 			)
 		)
-		(property "Footprint" "footprints:MSR421R"
+		(property "Footprint" "custom_comps:MSR421R"
 			(at 193.04 73.406 90)
 			(effects
@@
 			)
 		)
-		(property "Footprint" "KiCAD Parts:SOP65P490X110-8N"
+		(property "Footprint" "custom_comps:SOP65P490X110-8N"
 			(at 86.36 97.79 0)
 			(effects
@@
 			)
 		)
-		(property "Footprint" "footprints:ATGM336H"
+		(property "Footprint" "custom_comps:ATGM336H"
 			(at 144.78 76.2 0)
 			(effects
