File: pcb/esp32s3/ioexpander.kicad_sch (KiCad schematic)
At the start: 2 parts, among them U11 TCA9539RGER

Commit message: pcb kinda almost done!
Connections:
- net VDD renamed +3V3
Changed lines of the file:
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@@
 	)
 	(symbol
-		(lib_id "power:VDD")
+		(lib_id "power:+3V3")
 		(at 125.73 49.53 0)
 		(unit 1)
@@
 			)
 		)
-		(property "Value" "VDD"
+		(property "Value" "+3V3"
 			(at 125.73 44.45 0)
 			(effects
@@
 			)
 		)
-		(property "Description" "Power symbol creates a global label with name \"VDD\""
+		(property "Description" "Power symbol creates a global label with name \"+3V3\""
 			(at 125.73 49.53 0)
 			(effects
