File: pcb/esp32s3/untitled.kicad_sch (KiCad schematic)
At the start: 6 parts, among them U8 LSM303AGR

Commit message: Update PCB with new components and footprints
Parts:
- U8: footprint KiCAD Parts:PQFN50P200X200X100-12N -> custom_comps:PQFN50P200X200X100-12N
Changed lines of the file:
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@@
 			)
 		)
-		(property "Footprint" "KiCAD Parts:PQFN50P200X200X100-12N"
+		(property "Footprint" "custom_comps:PQFN50P200X200X100-12N"
 			(at 142.24 99.06 0)
 			(effects

Commit message: pcb kinda almost done!
Connections:
- net SCL: now also U8.1 (SCL/SPC)
- net SDA: now also U8.4 (SDA/SDI/SDO)
- net CS_XL: now reaches U8.2 (CS_XL)
- net CS_XL: now also R14.2
- net CS_MAG: now reaches U8.3 (CS_MAG)
- net CS_MAG: now also R15.2
Changed lines of the file:
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@@
+		)
+	)
+	(hierarchical_label "CS_MAG"
+		(shape input)
+		(at 43.18 31.75 270)
+		(fields_autoplaced yes)
+		(effects
+			(font
+				(size 1.27 1.27)
+			)
+			(justify right)
+		)
+	)
+	(hierarchical_label "CS_XL"
+		(shape input)
+		(at 29.21 31.75 270)
+		(fields_autoplaced yes)
+		(effects
+			(font
+				(size 1.27 1.27)
+			)
+			(justify right)
+		)
+	)
+	(hierarchical_label "SCL"
+		(shape input)
+		(at 119.38 99.06 180)
+		(fields_autoplaced yes)
+		(effects
+			(font
+				(size 1.27 1.27)
+			)
+			(justify right)
 		)
 	)
@@
 		)
 	)
-	(hierarchical_label "SCL"
-		(shape bidirectional)
-		(at 63.5 34.29 180)
+	(hierarchical_label "CS_MAG"
+		(shape input)
+		(at 119.38 93.98 180)
+		(fields_autoplaced yes)
+		(effects
+			(font
+				(size 1.27 1.27)
+			)
+			(justify right)
+		)
+	)
+	(hierarchical_label "CS_XL"
+		(shape input)
+		(at 119.38 91.44 180)
 		(fields_autoplaced yes)
 		(effects
@@
 	(hierarchical_label "SDA"
 		(shape bidirectional)
-		(at 78.74 34.29 180)
+		(at 119.38 104.14 180)
 		(fields_autoplaced yes)
 		(effects
@@
 		)
 	)
-	(netclass_flag ""
-		(length 2.54)
-		(shape round)
-		(at 43.18 31.75 180)
+	(hierarchical_label "SCL"
+		(shape bidirectional)
+		(at 63.5 34.29 270)
 		(fields_autoplaced yes)
 		(effects
@@
 				(size 1.27 1.27)
 			)
-			(justify right bottom)
-		)
-		(property "Netclass" "CS_MAG"
-			(at 43.8785 34.29 0)
-			(effects
-				(font
-					(size 1.27 1.27)
-					(italic yes)
-				)
-				(justify left)
-			)
+			(justify right)
 		)
 	)
-	(netclass_flag ""
-		(length 2.54)
-		(shape round)
-		(at 119.38 91.44 90)
+	(hierarchical_label "SDA"
+		(shape bidirectional)
+		(at 78.74 34.29 270)
+		(fields_autoplaced yes)
 		(effects
 			(font
 				(size 1.27 1.27)
 			)
-			(justify left bottom)
-		)
-		(property "Netclass" "CS_XL"
-			(at 109.728 91.44 0)
-			(effects
-				(font
-					(size 1.27 1.27)
-					(italic yes)
-				)
-				(justify left)
-			)
+			(justify right)
 		)
 	)
@@
 		(length 2.54)
 		(shape round)
-		(at 119.38 104.14 90)
-		(effects
-			(font
-				(size 1.27 1.27)
-			)
-			(justify left bottom)
-		)
-		(property "Netclass" "SDA"
-			(at 111.76 104.14 0)
-			(effects
-				(font
-					(size 1.27 1.27)
-					(italic yes)
-				)
-				(justify left)
-			)
-		)
-	)
-	(netclass_flag ""
-		(length 2.54)
-		(shape round)
-		(at 119.38 93.98 90)
-		(effects
-			(font
-				(size 1.27 1.27)
-			)
-			(justify left bottom)
-		)
-		(property "Netclass" "CS_MAG"
-			(at 108.204 93.98 0)
-			(effects
-				(font
-					(size 1.27 1.27)
-					(italic yes)
-				)
-				(justify left)
-			)
-		)
-	)
-	(netclass_flag ""
-		(length 2.54)
-		(shape round)
-		(at 29.21 31.75 180)
-		(fields_autoplaced yes)
-		(effects
-			(font
-				(size 1.27 1.27)
-			)
-			(justify right bottom)
-		)
-		(property "Netclass" "CS_XL"
-			(at 29.9085 34.29 0)
-			(effects
-				(font
-					(size 1.27 1.27)
-					(italic yes)
-				)
-				(justify left)
-			)
-		)
-	)
-	(netclass_flag ""
-		(length 2.54)
-		(shape round)
 		(at 78.74 31.75 270)
 		(effects
@@
 			(effects
 				(font
-					(size 1.27 1.27)
-					(italic yes)
-				)
-				(justify left)
-			)
-		)
-	)
-	(netclass_flag ""
-		(length 2.54)
-		(shape round)
-		(at 119.38 99.06 90)
-		(effects
-			(font
-				(size 1.27 1.27)
-			)
-			(justify left bottom)
-		)
-		(property "Netclass" "SCL"
-			(at 112.014 99.06 0)
-			(effects
-				(font
