File: pcb/stm32h7/display.kicad_sch (KiCad schematic)
At the start: 4 parts, among them J5 Conn_01x40_Socket

Commit message: fixed some wiring
Connections:
- net +3V3: no longer J5.1 (Pin_1)
- net LCD_BL renamed LCD_BL_CATHODE
- new net LCD_BL_ANODE: J5.1 (Pin_1)
Changed lines of the file:
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@@
-	)
-	(junction
-		(at 139.7 50.8)
-		(diameter 0)
-		(color 0 0 0 0)
 	)
 	(junction
@@
 	)
 	(junction
-		(at 146.05 88.9)
+		(at 143.51 52.07)
 		(diameter 0)
 		(color 0 0 0 0)
 	)
 	(junction
-		(at 139.7 48.26)
+		(at 139.7 53.34)
+		(diameter 0)
+		(color 0 0 0 0)
+	)
+	(junction
+		(at 146.05 88.9)
 		(diameter 0)
 		(color 0 0 0 0)
@@
 		(color 0 0 0 0)
 	)
-	(junction
-		(at 144.78 53.34)
-		(diameter 0)
-		(color 0 0 0 0)
-	)
 	(no_connect
 		(at 147.32 142.24)
@@
 	(wire
 		(pts
-			(xy 124.46 57.15) (xy 124.46 55.88)
+			(xy 116.84 57.15) (xy 116.84 55.88)
+		)
+		(stroke
+			(width 0)
+			(type default)
+		)
+	)
+	(wire
+		(pts
+			(xy 143.51 52.07) (xy 143.51 53.34)
 		)
 		(stroke
@@
 	(wire
 		(pts
-			(xy 147.32 50.8) (xy 144.78 50.8)
-		)
-		(stroke
-			(width 0)
-			(type default)
-		)
-	)
-	(wire
-		(pts
 			(xy 146.05 86.36) (xy 146.05 88.9)
 		)
@@
 	(wire
 		(pts
-			(xy 147.32 53.34) (xy 144.78 53.34)
-		)
-		(stroke
-			(width 0)
-			(type default)
-		)
-	)
-	(wire
-		(pts
 			(xy 139.7 35.56) (xy 139.7 38.1)
 		)
@@
 	(wire
 		(pts
-			(xy 119.38 53.34) (xy 144.78 53.34)
+			(xy 143.51 50.8) (xy 143.51 52.07)
 		)
 		(stroke
@@
 	(wire
 		(pts
-			(xy 139.7 48.26) (xy 139.7 50.8)
-		)
-		(stroke
-			(width 0)
-			(type default)
-		)
-	)
-	(wire
-		(pts
 			(xy 146.05 119.38) (xy 147.32 119.38)
 		)
@@
 	(wire
 		(pts
-			(xy 144.78 50.8) (xy 144.78 53.34)
+			(xy 139.7 38.1) (xy 139.7 53.34)
 		)
 		(stroke
@@
 	(wire
 		(pts
+			(xy 147.32 53.34) (xy 143.51 53.34)
+		)
+		(stroke
+			(width 0)
+			(type default)
+		)
+	)
+	(wire
+		(pts
 			(xy 139.7 132.08) (xy 139.7 147.32)
 		)
@@
 	(wire
 		(pts
-			(xy 147.32 48.26) (xy 139.7 48.26)
-		)
-		(stroke
-			(width 0)
-			(type default)
-		)
-	)
-	(wire
-		(pts
 			(xy 147.32 58.42) (xy 139.7 58.42)
 		)
@@
 	(wire
 		(pts
-			(xy 124.46 55.88) (xy 147.32 55.88)
+			(xy 116.84 55.88) (xy 147.32 55.88)
+		)
+		(stroke
+			(width 0)
+			(type default)
+		)
+	)
+	(wire
+		(pts
+			(xy 132.08 48.26) (xy 147.32 48.26)
 		)
 		(stroke
@@
 	(wire
 		(pts
-			(xy 135.89 59.69) (xy 135.89 50.8)
+			(xy 135.89 59.69) (xy 135.89 53.34)
+		)
+		(stroke
+			(width 0)
+			(type default)
+		)
+	)
+	(wire
+		(pts
+			(xy 139.7 53.34) (xy 139.7 58.42)
 		)
 		(stroke
@@
 	(wire
 		(pts
-			(xy 139.7 50.8) (xy 139.7 58.42)
-		)
-		(stroke
-			(width 0)
-			(type default)
-		)
-	)
-	(wire
-		(pts
-			(xy 135.89 50.8) (xy 139.7 50.8)
-		)
-		(stroke
-			(width 0)
-			(type default)
-		)
-	)
-	(wire
-		(pts
-			(xy 139.7 38.1) (xy 139.7 48.26)
+			(xy 135.89 53.34) (xy 139.7 53.34)
+		)
+		(stroke
+			(width 0)
+			(type default)
+		)
+	)
+	(wire
+		(pts
+			(xy 132.08 52.07) (xy 143.51 52.07)
+		)
+		(stroke
+			(width 0)
+			(type default)
+		)
+	)
+	(wire
+		(pts
+			(xy 143.51 50.8) (xy 147.32 50.8)
 		)
 		(stroke
@@
 		)
 	)
+	(hierarchical_label "LCD_BL_ANODE"
+		(shape input)
+		(at 132.08 48.26 180)
+		(fields_autoplaced yes)
+		(effects
+			(font
+				(size 1.27 1.27)
+			)
+			(justify right)
+		)
+	)
 	(hierarchical_label "LCD_G1"
 		(shape input)
@@
 		)
 	)
-	(hierarchical_label "LCD_BL"
-		(shape input)
-		(at 119.38 53.34 180)
+	(hierarchical_label "LCD_BL_CATHODE"
+		(shape input)
+		(at 132.08 52.07 180)
 		(fields_autoplaced yes)
 		(effects
@@
 	(symbol
 		(lib_id "power:GND")
-		(at 124.46 57.15 0)
+		(at 116.84 57.15 0)
 		(unit 1)
 		(exclude_from_sim no)
@@
 		(fields_autoplaced yes)
 		(property "Reference" "#PWR071"
-			(at 124.46 63.5 0)
+			(at 116.84 63.5 0)
 			(effects
 				(font
@@
 		)
 		(property "Value" "GND"
-			(at 124.46 62.23 0)
+			(at 116.84 62.23 0)
 			(effects
 				(font
@@
 		)
 		(property "Footprint" ""
-			(at 124.46 57.15 0)
+			(at 116.84 57.15 0)
 			(effects
 				(font
@@
 		)
 		(property "Datasheet" ""
-			(at 124.46 57.15 0)
+			(at 116.84 57.15 0)
 			(effects
 				(font
@@
 		)
 		(property "Description" "Power symbol creates a global label with name \"GND\" , ground"
-			(at 124.46 57.15 0)
+			(at 116.84 57.15 0)
 			(effects
 				(font

Commit message: finished pcb, ordered v0.3
Parts:
- R5: value 100 -> 100R
Changed lines of the file:
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@@
 			)
 		)
-		(property "Value" "100"
+		(property "Value" "100R"
 			(at 123.444 73.152 90)
 			(effects

Commit message: ugh.... 6 layer....
Connections:
- net +3V3: now also J5.36 (Pin_36); no longer J5.5 (Pin_5)
- net GND: now also J5.1 (Pin_1), J5.37 (Pin_37), J5.7 (Pin_7); no longer J5.34 (Pin_34), J5.4 (Pin_4), J5.40 (Pin_40)
- net LCD_B1: now also J5.24 (Pin_24), J5.25 (Pin_25); no longer J5.16 (Pin_16), J5.17 (Pin_17)
- net LCD_B2: now also J5.23 (Pin_23); no longer J5.18 (Pin_18)
- net LCD_B3: now also J5.22 (Pin_22); no longer J5.19 (Pin_19)
- net LCD_B4: now also J5.21 (Pin_21); no longer J5.20 (Pin_20)
- net LCD_B5: now also J5.20 (Pin_20); no longer J5.21 (Pin_21)
- net LCD_BL_ANODE: now also J5.40 (Pin_40); no longer J5.1 (Pin_1)
- net LCD_BL_CATHODE: now also J5.38 (Pin_38), J5.39 (Pin_39); no longer J5.2 (Pin_2), J5.3 (Pin_3)
- net LCD_CS: now also J5.30 (Pin_30); no longer J5.11 (Pin_11)
- net LCD_DE: now also J5.28 (Pin_28); no longer J5.13 (Pin_13)
- net LCD_G0: now also J5.19 (Pin_19); no longer J5.22 (Pin_22)
- net LCD_G1: now also J5.18 (Pin_18); no longer J5.23 (Pin_23)
- net LCD_G2: now also J5.17 (Pin_17); no longer J5.24 (Pin_24)
- net LCD_G3: now also J5.16 (Pin_16); no longer J5.25 (Pin_25)
- net LCD_G4: now also J5.15 (Pin_15); no longer J5.26 (Pin_26)
- net LCD_G5: now also J5.14 (Pin_14); no longer J5.27 (Pin_27)
- net LCD_HSYNC: now also J5.26 (Pin_26); no longer J5.15 (Pin_15)
- net LCD_MOSI: now also J5.32 (Pin_32); no longer J5.9 (Pin_9)
- net LCD_R1: now also J5.12 (Pin_12), J5.13 (Pin_13); no longer J5.28 (Pin_28), J5.29 (Pin_29)
- net LCD_R2: now also J5.11 (Pin_11); no longer J5.30 (Pin_30)
- net LCD_R3: now also J5.10 (Pin_10); no longer J5.31 (Pin_31)
- net LCD_R4: now also J5.9 (Pin_9); no longer J5.32 (Pin_32)
- net LCD_R5: now also J5.8 (Pin_8); no longer J5.33 (Pin_33)
- net LCD_RST: now also J5.35 (Pin_35); no longer J5.6 (Pin_6)
- net LCD_SCK: now also J5.31 (Pin_31); no longer J5.10 (Pin_10)
- net LCD_VSYNC: now also J5.27 (Pin_27); no longer J5.14 (Pin_14)
- net at R5.2: now also J5.29 (Pin_29); no longer J5.12 (Pin_12)
Changed lines of the file:
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@@
 	(symbol
 		(lib_id "Connector:Conn_01x40_Socket")
-		(at 152.4 96.52 0)
+		(at 152.4 97.79 0)
 		(unit 1)
 		(exclude_from_sim no)
@@
 		(fields_autoplaced yes)
 		(property "Reference" "J5"
-			(at 154.94 96.5199 0)
+			(at 154.94 99.0601 0)
 			(effects
 				(font
@@
 		)
 		(property "Value" "Conn_01x40_Socket"
-			(at 154.94 99.0599 0)
+			(at 154.94 96.5201 0)
 			(effects
 				(font
@@
 		)
 		(property "Footprint" "Connector_FFC-FPC:Hirose_FH12-40S-0.5SH_1x40-1MP_P0.50mm_Horizontal"
-			(at 152.4 96.52 0)
+			(at 152.4 99.06 0)
 			(effects
 				(font
@@
 		)
 		(property "Datasheet" "~"
-			(at 152.4 96.52 0)
+			(at 152.4 99.06 0)
 			(effects
 				(font
@@
 		)
 		(property "Description" "Generic connector, single row, 01x40, script generated"
-			(at 152.4 96.52 0)
+			(at 152.4 99.06 0)
 			(effects
 				(font
