File: pcb/stm32h7/stm32h7.kicad_sch (KiCad schematic)
At the start: 39 parts, among them J6 Test Pads, SW1 SW_Push, SW2 SW_Push, SW3 SW_Push, U1 STM32H743VGTx, U11 TPS61169DCKR, U9 MT25QUxxxxxx1xW7, Y1 25MHz

Commit message: finished pcb, ordered v0.3
Parts:
- C4, C5: value 3.9pF -> 8pF
- D3: value NSR0240 -> MBR0540
Other:
- moved on the sheet: C4, C5, Y1
Changed lines of the file:
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@@
 	)
 	(junction
-		(at 26.67 87.63)
+		(at 25.4 87.63)
 		(diameter 0)
 		(color 0 0 0 0)
@@
 	)
 	(junction
-		(at 35.56 80.01)
+		(at 34.29 80.01)
 		(diameter 0)
 		(color 0 0 0 0)
@@
 	)
 	(junction
-		(at 41.91 93.98)
-		(diameter 0)
-		(color 0 0 0 0)
-	)
-	(junction
 		(at 165.1 102.87)
 		(diameter 0)
@@
 	)
 	(junction
-		(at 35.56 101.6)
+		(at 34.29 101.6)
 		(diameter 0)
 		(color 0 0 0 0)
@@
 	(wire
 		(pts
-			(xy 41.91 100.33) (xy 41.91 101.6)
+			(xy 40.64 100.33) (xy 40.64 101.6)
 		)
 		(stroke
@@
 	(wire
 		(pts
-			(xy 35.56 80.01) (xy 35.56 88.9)
+			(xy 34.29 80.01) (xy 34.29 88.9)
 		)
 		(stroke
@@
 	(wire
 		(pts
-			(xy 35.56 101.6) (xy 35.56 102.87)
+			(xy 34.29 101.6) (xy 34.29 102.87)
 		)
 		(stroke
@@
 	(wire
 		(pts
-			(xy 41.91 93.98) (xy 43.18 93.98)
-		)
-		(stroke
-			(width 0)
-			(type default)
-		)
-	)
-	(wire
-		(pts
-			(xy 35.56 78.74) (xy 35.56 80.01)
+			(xy 34.29 78.74) (xy 34.29 80.01)
 		)
 		(stroke
@@
 	(wire
 		(pts
-			(xy 35.56 101.6) (xy 41.91 101.6)
+			(xy 34.29 101.6) (xy 40.64 101.6)
 		)
 		(stroke
@@
 	(wire
 		(pts
-			(xy 41.91 93.98) (xy 41.91 95.25)
+			(xy 40.64 93.98) (xy 40.64 95.25)
 		)
 		(stroke
@@
 	(wire
 		(pts
-			(xy 39.37 93.98) (xy 41.91 93.98)
+			(xy 38.1 93.98) (xy 40.64 93.98)
 		)
 		(stroke
@@
 	(wire
 		(pts
-			(xy 26.67 87.63) (xy 25.4 87.63)
+			(xy 25.4 87.63) (xy 24.13 87.63)
 		)
 		(stroke
@@
 	(wire
 		(pts
-			(xy 26.67 87.63) (xy 26.67 93.98)
+			(xy 25.4 87.63) (xy 25.4 93.98)
 		)
 		(stroke
@@
 	(wire
 		(pts
-			(xy 35.56 99.06) (xy 35.56 101.6)
+			(xy 34.29 99.06) (xy 34.29 101.6)
 		)
 		(stroke
@@
 	(wire
 		(pts
-			(xy 31.75 93.98) (xy 26.67 93.98)
+			(xy 30.48 93.98) (xy 25.4 93.98)
 		)
 		(stroke
@@
 	(wire
 		(pts
-			(xy 26.67 80.01) (xy 26.67 81.28)
+			(xy 25.4 80.01) (xy 25.4 81.28)
 		)
 		(stroke
@@
 	(wire
 		(pts
-			(xy 26.67 86.36) (xy 26.67 87.63)
+			(xy 25.4 86.36) (xy 25.4 87.63)
 		)
 		(stroke
@@
 	(wire
 		(pts
-			(xy 26.67 80.01) (xy 35.56 80.01)
+			(xy 25.4 80.01) (xy 34.29 80.01)
 		)
 		(stroke
@@
 	(global_label "PH1"
 		(shape input)
-		(at 43.18 93.98 0)
+		(at 40.64 93.98 0)
 		(fields_autoplaced yes)
 		(effects
@@
 		)
 		(property "Intersheetrefs" "${INTERSHEET_REFS}"
-			(at 49.9752 93.98 0)
+			(at 47.4352 93.98 0)
 			(effects
 				(font
@@
 	(global_label "PH0"
 		(shape input)
-		(at 25.4 87.63 180)
+		(at 24.13 87.63 180)
 		(fields_autoplaced yes)
 		(effects
@@
 		)
 		(property "Intersheetrefs" "${INTERSHEET_REFS}"
-			(at 18.6048 87.63 0)
+			(at 17.3348 87.63 0)
 			(effects
 				(font
@@
 			)
 		)
-		(property "Value" "NSR0240"
+		(property "Value" "MBR0540"
 			(at 274.32 21.844 0)
 			(effects
@@
 	(symbol
 		(lib_id "Device:Crystal_GND24")
-		(at 35.56 93.98 0)
+		(at 34.29 93.98 0)
 		(unit 1)
 		(exclude_from_sim no)
@@
 		(dnp no)
 		(property "Reference" "Y1"
-			(at 24.638 96.52 0)
+			(at 23.368 96.52 0)
 			(effects
 				(font
@@
 		)
 		(property "Value" "25MHz"
-			(at 24.638 99.06 0)
+			(at 23.368 99.06 0)
 			(effects
 				(font
@@
 		)
 		(property "Footprint" "Crystal:Crystal_SMD_2016-4Pin_2.0x1.6mm"
-			(at 35.56 93.98 0)
+			(at 34.29 93.98 0)
 			(effects
 				(font
@@
 		)
 		(property "Datasheet" "~"
-			(at 35.56 93.98 0)
+			(at 34.29 93.98 0)
 			(effects
 				(font
@@
 		)
 		(property "Description" "Four pin crystal, GND on pins 2 and 4"
-			(at 35.56 93.98 0)
+			(at 34.29 93.98 0)
 			(effects
 				(font
@@
 	(symbol
 		(lib_id "power:GND")
-		(at 35.56 78.74 180)
+		(at 34.29 78.74 180)
 		(unit 1)
 		(exclude_from_sim no)
@@
 		(fields_autoplaced yes)
 		(property "Reference" "#PWR013"
-			(at 35.56 72.39 0)
+			(at 34.29 72.39 0)
 			(effects
 				(font
@@
 		)
 		(property "Value" "GND"
-			(at 35.56 73.66 0)
+			(at 34.29 73.66 0)
 			(effects
 				(font
@@
 		)
 		(property "Footprint" ""
-			(at 35.56 78.74 0)
+			(at 34.29 78.74 0)
 			(effects
 				(font
@@
 		)
 		(property "Datasheet" ""
-			(at 35.56 78.74 0)
+			(at 34.29 78.74 0)
 			(effects
 				(font
@@
 		)
 		(property "Description" "Power symbol creates a global label with name \"GND\" , ground"
-			(at 35.56 78.74 0)
+			(at 34.29 78.74 0)
 			(effects
 				(font
@@
 	(symbol
 		(lib_id "Device:C_Small")
-		(at 26.67 83.82 0)
+		(at 25.4 83.82 0)
 		(unit 1)
 		(exclude_from_sim no)
@@
 		(fields_autoplaced yes)
 		(property "Reference" "C5"
-			(at 29.21 82.5562 0)
+			(at 27.94 82.5562 0)
 			(effects
 				(font
@@
 			)
 		)
-		(property "Value" "3.9pF"
-			(at 29.21 85.0962 0)
+		(property "Value" "8pF"
+			(at 27.94 85.0962 0)
 			(effects
 				(font
@@
 		)
 		(property "Footprint" "Capacitor_SMD:C_0402_1005Metric"
-			(at 26.67 83.82 0)
+			(at 25.4 83.82 0)
 			(effects
 				(font
@@
 		)
 		(property "Datasheet" "~"
-			(at 26.67 83.82 0)
+			(at 25.4 83.82 0)
 			(effects
 				(font
@@
 		)
 		(property "Description" "Unpolarized capacitor, small symbol"
-			(at 26.67 83.82 0)
+			(at 25.4 83.82 0)
 			(effects
 				(font
@@
 	(symbol
 		(lib_id "Device:C_Small")
-		(at 41.91 97.79 0)
+		(at 40.64 97.79 0)
 		(unit 1)
 		(exclude_from_sim no)
@@
 		(fields_autoplaced yes)
 		(property "Reference" "C4"
-			(at 44.45 96.5262 0)
+			(at 43.18 96.5262 0)
 			(effects
 				(font
@@
 			)
 		)
-		(property "Value" "3.9pF"
-			(at 44.45 99.0662 0)
+		(property "Value" "8pF"
+			(at 43.18 99.0662 0)
 			(effects
 				(font
@@
 		)
 		(property "Footprint" "Capacitor_SMD:C_0402_1005Metric"
-			(at 41.91 97.79 0)
+			(at 40.64 97.79 0)
 			(effects
 				(font
@@
 		)
 		(property "Datasheet" "~"
-			(at 41.91 97.79 0)
+			(at 40.64 97.79 0)
 			(effects
 				(font
@@
 		)
 		(property "Description" "Unpolarized capacitor, small symbol"
-			(at 41.91 97.79 0)
+			(at 40.64 97.79 0)
 			(effects
 				(font
@@
 	(symbol
 		(lib_id "power:GND")
-		(at 35.56 102.87 0)
+		(at 34.29 102.87 0)
 		(unit 1)
 		(exclude_from_sim no)
@@
 		(fields_autoplaced yes)
 		(property "Reference" "#PWR010"
-			(at 35.56 109.22 0)
+			(at 34.29 109.22 0)
 			(effects
 				(font
@@
 		)
 		(property "Value" "GND"
-			(at 35.56 107.95 0)
+			(at 34.29 107.95 0)
 			(effects
 				(font
@@
 		)
 		(property "Footprint" ""
-			(at 35.56 102.87 0)
+			(at 34.29 102.87 0)
 			(effects
 				(font
@@
 		)
 		(property "Datasheet" ""
-			(at 35.56 102.87 0)
+			(at 34.29 102.87 0)
 			(effects
 				(font
@@
 		)
 		(property "Description" "Power symbol creates a global label with name \"GND\" , ground"
-			(at 35.56 102.87 0)
+			(at 34.29 102.87 0)
 			(effects
 				(font

Commit message: everything is connected....
Connections:
- net +3V3: no longer SW1.2
- net BTN: now also U1.9 (PC15); no longer U1.33 (PC5)
- net GND: now also U1.33 (PC5); no longer U1.9 (PC15)
- net GPS_RXD: now also U1.98 (PE1); no longer U1.97 (PE0)
- net GPS_TXD: now also U1.97 (PE0); no longer U1.98 (PE1)
- net VCC: now also SW1.2
Changed lines of the file:
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@@
 	)
 	(junction
+		(at 177.8 142.24)
+		(diameter 0)
+		(color 0 0 0 0)
+	)
+	(junction
 		(at 156.21 185.42)
 		(diameter 0)
@@
 	)
 	(junction
-		(at 177.8 140.97)
-		(diameter 0)
-		(color 0 0 0 0)
-	)
-	(junction
-		(at 165.1 163.83)
-		(diameter 0)
-		(color 0 0 0 0)
-	)
-	(junction
 		(at 228.6 31.75)
 		(diameter 0)
@@
 	)
 	(junction
+		(at 165.1 140.97)
+		(diameter 0)
+		(color 0 0 0 0)
+	)
+	(junction
 		(at 86.36 110.49)
 		(diameter 0)
@@
 	(wire
 		(pts
-			(xy 149.86 166.37) (xy 165.1 166.37)
+			(xy 149.86 166.37) (xy 173.99 166.37)
 		)
 		(stroke
@@
 	(wire
 		(pts
-			(xy 165.1 135.89) (xy 165.1 148.59)
+			(xy 165.1 135.89) (xy 165.1 140.97)
 		)
 		(stroke
@@
 	(wire
 		(pts
+			(xy 173.99 142.24) (xy 177.8 142.24)
+		)
+		(stroke
+			(width 0)
+			(type default)
+		)
+	)
+	(wire
+		(pts
 			(xy 203.2 104.14) (xy 207.01 104.14)
 		)
@@
 		)
 	)
+	(wire
+		(pts
+			(xy 173.99 166.37) (xy 173.99 142.24)
+		)
+		(stroke
+			(width 0)
+			(type default)
+		)
+	)
 	(polyline
 		(pts
@@
 	(wire
 		(pts
-			(xy 177.8 140.97) (xy 177.8 138.43)
-		)
-		(stroke
-			(width 0)
-			(type default)
-		)
-	)
-	(wire
-		(pts
 			(xy 149.86 163.83) (xy 165.1 163.83)
 		)
@@
 	(wire
 		(pts
+			(xy 170.18 46.99) (xy 170.18 176.53)
+		)
+		(stroke
+			(width 0)
+			(type default)
+		)
+	)
+	(wire
+		(pts
 			(xy 165.1 102.87) (xy 165.1 115.57)
 		)
@@
 	(wire
 		(pts
-			(xy 149.86 140.97) (xy 177.8 140.97)
+			(xy 100.33 163.83) (xy 100.33 160.02)
 		)
 		(stroke
@@
 	(wire
 		(pts
-			(xy 100.33 163.83) (xy 100.33 160.02)
+			(xy 219.71 85.09) (xy 205.74 85.09)
 		)
 		(stroke
@@
 	(wire
 		(pts
-			(xy 219.71 85.09) (xy 205.74 85.09)
+			(xy 165.1 133.35) (xy 165.1 135.89)
 		)
 		(stroke
@@
 	(wire
 		(pts
-			(xy 165.1 133.35) (xy 165.1 135.89)
+			(xy 30.48 143.51) (xy 34.29 143.51)
 		)
 		(stroke
@@
 	(wire
 		(pts
-			(xy 30.48 143.51) (xy 34.29 143.51)
+			(xy 149.86 133.35) (xy 165.1 133.35)
 		)
 		(stroke
@@
 	(wire
 		(pts
-			(xy 149.86 133.35) (xy 165.1 133.35)
+			(xy 165.1 151.13) (xy 165.1 156.21)
 		)
 		(stroke
@@
 	(wire
 		(pts
-			(xy 165.1 151.13) (xy 165.1 156.21)
+			(xy 149.86 140.97) (xy 165.1 140.97)
 		)
 		(stroke
@@
 	(wire
 		(pts
-			(xy 177.8 144.78) (xy 177.8 140.97)
+			(xy 177.8 138.43) (xy 177.8 142.24)
 		)
 		(stroke
@@
 	(wire
 		(pts
-			(xy 170.18 46.99) (xy 170.18 176.53)
-		)
-		(stroke
-			(width 0)
-			(type default)
-		)
-	)
-	(wire
-		(pts
 			(xy 149.86 102.87) (xy 165.1 102.87)
 		)
@@
 		)
 	)
-	(wire
+	(polyline
 		(pts
-			(xy 165.1 163.83) (xy 165.1 166.37)
+			(xy 177.0288 12.0241) (xy 177.033 12.0241)
 		)
 		(stroke
@@
 		)
 	)
-	(polyline
+	(wire
 		(pts
-			(xy 177.0288 12.0241) (xy 177.033 12.0241)
+			(xy 149.86 41.91) (xy 165.1 41.91)
 		)
 		(stroke
@@
 	(wire
 		(pts
-			(xy 149.86 41.91) (xy 165.1 41.91)
+			(xy 25.4 80.01) (xy 34.29 80.01)
 		)
 		(stroke
@@
 	(wire
 		(pts
-			(xy 25.4 80.01) (xy 34.29 80.01)
+			(xy 124.46 21.59) (xy 124.46 34.29)
 		)
 		(stroke
@@
 	(wire
 		(pts
-			(xy 124.46 21.59) (xy 124.46 34.29)
+			(xy 165.1 140.97) (xy 165.1 148.59)
 		)
 		(stroke
@@
 	(wire
 		(pts
+			(xy 177.8 142.24) (xy 177.8 144.78)
+		)
+		(stroke
+			(width 0)
+			(type default)
+		)
+	)
+	(wire
+		(pts
 			(xy 153.67 24.13) (xy 153.67 21.59)
 		)
@@
 	(wire
 		(pts
+			(xy 177.8 156.21) (xy 177.8 154.94)
+		)
+		(stroke
+			(width 0)
+			(type default)
+		)
+	)
+	(wire
+		(pts
 			(xy 165.1 158.75) (xy 165.1 161.29)
 		)
@@
 	(global_label "GPS_TXD"
 		(shape input)
-		(at 106.68 67.31 180)
+		(at 106.68 64.77 180)
 		(fields_autoplaced yes)
 		(effects
@@
 		)
 		(property "Intersheetrefs" "${INTERSHEET_REFS}"
-			(at 95.5306 67.31 0)
+			(at 95.5306 64.77 0)
 			(effects
 				(font
@@
 	(global_label "GPS_RXD"
 		(shape input)
-		(at 106.68 64.77 180)
+		(at 106.68 67.31 180)
 		(fields_autoplaced yes)
 		(effects
@@
 		)
 		(property "Intersheetrefs" "${INTERSHEET_REFS}"
-			(at 95.2282 64.77 0)
+			(at 95.2282 67.31 0)
 			(effects
 				(font
@@
 	)
 	(symbol
+		(lib_id "power:VCC")
+		(at 177.8 156.21 180)
+		(unit 1)
+		(exclude_from_sim no)
+		(in_bom yes)
+		(on_board yes)
+		(dnp no)
+		(fields_autoplaced yes)
+		(property "Reference" "#PWR069"
+			(at 177.8 152.4 0)
+			(effects
+				(font
+					(size 1.27 1.27)
+				)
+				(hide yes)
+			)
+		)
+		(property "Value" "VCC"
+			(at 177.8 161.29 0)
+			(effects
+				(font
+					(size 1.27 1.27)
+				)
+			)
+		)
+		(property "Footprint" ""
+			(at 177.8 156.21 0)
+			(effects
+				(font
+					(size 1.27 1.27)
+				)
+				(hide yes)
+			)
+		)
+		(property "Datasheet" ""
+			(at 177.8 156.21 0)
+			(effects
+				(font
+					(size 1.27 1.27)
+				)
+				(hide yes)
+			)
+		)
+		(property "Description" "Power symbol creates a global label with name \"VCC\""
+			(at 177.8 156.21 0)
+			(effects
+				(font
+					(size 1.27 1.27)
+				)
+				(hide yes)
+			)
+		)
+		(pin "1"
+		)
+		(instances
+			(project "stm32h7"
+				(path "/834edf73-57a5-43b4-ab36-0b077e93e6d5"
+					(reference "#PWR069")
+					(unit 1)
+				)
+			)
+		)
+	)
+	(symbol
 		(lib_id "power:+3V3")
 		(at 124.46 20.32 0)
@@
 					(unit 1)
 				)
-			)
-		)
-	)
-	(symbol
-		(lib_id "power:+3V3")
-		(at 177.8 154.94 180)
-		(unit 1)
-		(exclude_from_sim no)
-		(in_bom yes)
-		(on_board yes)
-		(dnp no)
-		(fields_autoplaced yes)
-		(property "Reference" "#PWR069"
-			(at 177.8 151.13 0)
-			(effects
-				(font
-					(size 1.27 1.27)
-				)
-				(hide yes)
-			)
-		)
-		(property "Value" "+3V3"
-			(at 177.8 160.02 0)
-			(effects
-				(font
-					(size 1.27 1.27)
-				)
-			)
-		)
-		(property "Footprint" ""
-			(at 177.8 154.94 0)
-			(effects
-				(font
-					(size 1.27 1.27)
-				)
-				(hide yes)
-			)
-		)
-		(property "Datasheet" ""
-			(at 177.8 154.94 0)
-			(effects
-				(font
-					(size 1.27 1.27)
-				)
-				(hide yes)
-			)
-		)
-		(property "Description" "Power symbol creates a global label with name \"+3V3\""
-			(at 177.8 154.94 0)
-			(effects
-				(font
-					(size 1.27 1.27)
-				)
-				(hide yes)
-			)
-		)
-		(pin "1"
-		)
-		(instances
-			(project "stm32h7"
-				(path "/834edf73-57a5-43b4-ab36-0b077e93e6d5"
-					(reference "#PWR069")
-					(unit 1)
-				)
