File: pcb/stm32h7/untitled.kicad_sch (KiCad schematic)
At the start: 6 parts, among them U8 LSM303AGR

Commit message: is it finally done or am i going insane
Parts:
- removed R14: 10K, Resistor_SMD:R_0402_1005Metric, symbol Device:R_Small
- added C38: 100nF, Capacitor_SMD:C_0402_1005Metric, symbol Device:C_Small
- added C39: 10uF, Capacitor_SMD:C_0402_1005Metric, symbol Device:C_Small
Connections:
- net CS_XL is gone; now on net CS_MAG: U8.2 (CS_XL)
- net +3V3: now also C38.2, C39.2
- net GND: now also C38.1, C39.1
