File: pcb/stm32h7/stm32h7.kicad_pcb (KiCad board)
At the start: 4 copper layers, 59.7 x 58.9 mm, 93 parts, among them J1 USB_C_Receptacle_USB2.0_14P, J2 Battery, J3 GPS_ANT, J4 Conn_Coaxial, J5 Conn_01x40_Socket, J6 Test Pads, Q1 DMG3414U, Q1_Xtal1 32.0MHz, SW1 SW_Push, SW2 SW_Push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

Commit message: ugh.... 6 layer....
Parts:
- C1, C2: value 220nF -> 200nF
- D3: value NSR0240 -> MBR0540
- R5: value 100 -> 100R
Connections:
- J5 pad 1: BL_ANODE -> GND
- J5 pad 10: SCK -> LCD_R3
- J5 pad 11: LCD_CS -> LCD_R2
- J5 pad 12: Net-(J5-Pin_12) -> LCD_R1
- J5 pad 13: LCD_DE -> LCD_R1
- J5 pad 14: LCD_VSYNC -> LCD_G5
- J5 pad 15: LCD_HSYNC -> LCD_G4
- J5 pad 16: LCD_B1 -> LCD_G3
- J5 pad 17: LCD_B1 -> LCD_G2
- J5 pad 18: LCD_B2 -> LCD_G1
- J5 pad 19: LCD_B3 -> LCD_G0
- J5 pad 2: BL_CATHODE -> unconnected-(J5-Pin_2-Pad2)
- J5 pad 20: LCD_B4 -> LCD_B5
- J5 pad 21: LCD_B5 -> LCD_B4
- J5 pad 22: LCD_G0 -> LCD_B3
- J5 pad 23: LCD_G1 -> LCD_B2
- J5 pad 24: LCD_G2 -> LCD_B1
- J5 pad 25: LCD_G3 -> LCD_B1
- J5 pad 26: LCD_G4 -> LCD_HSYNC
- J5 pad 27: LCD_G5 -> LCD_VSYNC
- J5 pad 28: LCD_R1 -> LCD_DE
- J5 pad 29: LCD_R1 -> Net-(J5-Pin_29)
- J5 pad 3: BL_CATHODE -> unconnected-(J5-Pin_3-Pad3)
- J5 pad 30: LCD_R2 -> LCD_CS
- J5 pad 31: LCD_R3 -> SCK
- J5 pad 32: LCD_R4 -> MOSI
- J5 pad 33: LCD_R5 -> unconnected-(J5-Pin_33-Pad33)
- J5 pad 34: GND -> unconnected-(J5-Pin_34-Pad34)
- J5 pad 35: unconnected-(J5-Pin_35-Pad35) -> LCD_RST
- J5 pad 36: unconnected-(J5-Pin_36-Pad36) -> +3V3
- J5 pad 37: unconnected-(J5-Pin_37-Pad37) -> GND
- J5 pad 38: unconnected-(J5-Pin_38-Pad38) -> BL_CATHODE
- J5 pad 39: unconnected-(J5-Pin_39-Pad39) -> BL_CATHODE
- J5 pad 4: GND -> unconnected-(J5-Pin_4-Pad4)
- J5 pad 40: GND -> BL_ANODE
- J5 pad 5: +3V3 -> unconnected-(J5-Pin_5-Pad5)
- J5 pad 6: LCD_RST -> unconnected-(J5-Pin_6-Pad6)
- J5 pad 7: unconnected-(J5-Pin_7-Pad7) -> GND
- J5 pad 8: unconnected-(J5-Pin_8-Pad8) -> LCD_R5
- J5 pad 9: MOSI -> LCD_R4
- R5 pad 2: Net-(J5-Pin_12) -> Net-(J5-Pin_29)
Routing:
- net SCL: track 99.0 -> 3.49 mm, vias 9 -> 0
- net BTN: track 89.4 -> 0.00 mm, vias 6 -> 0
- net SDA: track 68.0 -> 3.43 mm, vias 5 -> 0
- net LDO_EN: track 71.8 -> 10.5 mm, vias 6 -> 2
- net LoRa_NSS: track 46.7 -> 0.00 mm, vias 4 -> 0
- net MISO: track 43.4 -> 0.00 mm, vias 2 -> 0
- net GND: track 106.5 -> 63.5 mm, vias 494 -> 427
- net VBUS: track 68.3 -> 26.4 mm, vias 4 -> 0
- net LoRa_DIO1: track 39.7 -> 0.00 mm, vias 4 -> 0
- net LoRa_RST: track 39.5 -> 0.00 mm, vias 6 -> 0
- net LoRa_BUSY: track 39.4 -> 0.00 mm, vias 4 -> 0
- net FG_NALERT: track 39.1 -> 0.00 mm, vias 2 -> 0
- net SCK: track 61.4 -> 23.1 mm, vias 4 -> 2
- net NRST: track 39.0 -> 6.67 mm, vias 2 -> 0
- net Net-(J5-Pin_29): track 0.00 -> 32.1 mm, vias 0 -> 2
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- added copper zone on In4.Cu, net GND
Other:
- copper layers 4 -> 6

Commit message: everything is connected....
Connections:
- SW1 pad 2: +3V3 -> VCC
- U1 pad 33: BTN -> GND
- U1 pad 9: GND -> BTN
- U1 pad 97: GPS_RXD -> GPS_TXD
- U1 pad 98: GPS_TXD -> GPS_RXD
Routing:
- net BTN: track 0.00 -> 76.7 mm, vias 0 -> 5
- net SDA: track 3.43 -> 62.3 mm, vias 0 -> 3
- net SCL: track 3.49 -> 61.2 mm, vias 0 -> 3
- net LDO_EN: track 10.5 -> 64.0 mm, vias 2 -> 5
- net FG_NALERT: track 0.00 -> 39.3 mm, vias 0 -> 2
- net VBUS: track 26.4 -> 63.9 mm, vias 0 -> 2
- net MISO: track 0.00 -> 35.7 mm, vias 0 -> 3
- net LoRa_RST: track 0.00 -> 33.8 mm, vias 0 -> 2
- net LoRa_DIO1: track 0.00 -> 33.5 mm, vias 0 -> 2
- net LoRa_BUSY: track 0.00 -> 33.3 mm, vias 0 -> 2
- net LoRa_NSS: track 0.00 -> 27.5 mm, vias 0 -> 2
- net USB_D-: track 0.00 -> 27.3 mm
- net USB_D+: track 0.00 -> 27.3 mm
- net INT_MAG: track 0.00 -> 23.4 mm
- net NRST: track 6.67 -> 28.0 mm, vias 0 -> 4
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- added copper zone on In3.Cu, net GND

Commit message: finishing touches, sent to jlcpcb
Parts:
- moved SW1 0.35 mm to (142.2, 94.3)
Routing:
- net LCD_G2: track 20.7 -> 41.6 mm
- net QSPI_D2: track 6.78 -> 25.9 mm
- net LCD_B1: track 20.8 -> 39.2 mm
- net LCD_G5: track 21.5 -> 38.5 mm
- net LCD_G4: track 21.2 -> 38.1 mm
- net LCD_B4: track 23.7 -> 38.6 mm
- net LCD_G1: track 24.2 -> 38.9 mm
- net LCD_B5: track 24.8 -> 38.9 mm
- net LCD_R5: track 24.8 -> 38.1 mm
- net LCD_G0: track 29.2 -> 38.9 mm
- net QSPI_NCS: track 17.8 -> 27.2 mm
- net LCD_B2: track 30.8 -> 38.7 mm
- net QSPI_D3: track 19.7 -> 27.2 mm
- net LCD_R4: track 32.4 -> 38.1 mm
- net QSPI_CLK: track 22.8 -> 27.5 mm
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Other:
- board text added: "Festival Tracker v0.4 Big Z and Lil T Productions"
- board text removed: "Festival Tracker v0.3 Big Z and Lil T Productions"
- board text removed: "It is not the critic who counts; not the man who points out how the strong man stumbles, or where the doer of deeds could have done them better. The credit belongs to the man who is actually in the arena, whose face is marred by dust and sweat and blood; who strives valiantly; who errs, who comes short again and again, because there is no effort without error and shortcoming; but who does actuall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"
